Commit message: milestone - working tricycly with mimicd rear wheel.

File: curio_description/urdf/double_tricycle.urdf (robot description, URDF)
Before this commit: robot dtricycle_drive, 8 links, 7 joints
Links:
- link wheel_rear_link: geometry collision cylinder length=0.08 radius=0.32; visual cylinder length=0.08 radius=0.32
