Commit message: model showing up in rviz and gazebo now

File: curio_description/urdf/curio.urdf (robot description, URDF)
Before this commit: robot curio, 3 links, 2 joints
Links:
- link body_box_link: geometry collision box size=${body_box_length} ${body_box_width} ${body_box_depth}; visual mesh filename=file://$(find curio_description)/meshes/bases/body_box.stl
- link diff_brace_link: geometry collision box size=0.200 0.015 0.015; visual mesh filename=file://$(find curio_description)/meshes/bases/differential.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

File: curio_description/urdf/curio_laser.xacro (robot description, xacro)
@@ -37,5 +37,5 @@
                 <origin rpy="0 0 0" xyz="0 0 0" />
                 <geometry>
-                    <mesh filename="package://curio_description/meshes/sensors/rplidar_a1_assembly_low.stl" />
+                    <mesh filename="file://$(find curio_description)/meshes/sensors/rplidar_a1_assembly_low.stl" />
                 </geometry>
                 <material name="white" />

Commit message: loading curio and maze world into gazebo!

File: curio_description/urdf/curio.urdf (robot description, URDF)
Before this commit: robot curio, 3 links, 2 joints
Links:
- added link base_footprint
- link base_link: geometry collision box size=0.01 0.01 0.01; visual box size=0.01 0.01 0.01
Joints:
- added joint base_joint: type fixed, parent base_footprint, child base_link, origin xyz=0 0 0 rpy=0 0 0, axis 0 0 1
